Commit message: finalize robot sketch

File: urdf/differential_robot.xacro (robot description, xacro)
@@ -3,6 +3,6 @@
   <!-- ========================== Properties ========================== -->
   <xacro:property name="wheel_d" value="0.072" />
-  <xacro:property name="wheel_r" value="${wheel_d/2.0}" /> <!-- back wheel radius -->
-  <xacro:property name="wheel_w" value="0.008" /> <!-- wheel width -->
+  <xacro:property name="wheel_r" value="${wheel_d/2.0}" />
+  <xacro:property name="wheel_w" value="0.008" />
   <xacro:property name="base_radius" value="0.175" />
   <xacro:property name="base_thickness" value="0.02" />
@@ -15,9 +15,15 @@
   <xacro:property name="passive_wheel_r" value="0.02" />
   <xacro:property name="passive_wheel_w" value="0.01" />
+  <!-- Mass properties -->
+  <xacro:property name="mass_head" value="0.02" /> <!-- 20g -->
+  <xacro:property name="mass_base" value="0.1" />  <!-- 100g -->
+  <xacro:property name="mass_back_wheel" value="0.025" /> <!-- 25g -->
+  <xacro:property name="mass_passive_holder" value="0.015" /> <!-- 15g -->
+  <xacro:property name="mass_passive_wheel" value="0.01" /> <!-- 10g -->
   <material name="wheel_black">
     <color rgba="0.05 0.05 0.05 1.0" />
   </material>
   <!-- ========================== Links ========================== -->
-  <link name="base_footprint" /> <!-- dummy link -->
+  <link name="base_footprint" />
   <link name="base_link">
     <visual>
@@ -30,6 +36,6 @@
     </visual>
     <inertial>
-      <mass value="5.0" />
-      <inertia ixx="0.1" ixy="0.0" ixz="0.0" iyy="0.1" iyz="0.0" izz="0.1" />
+      <mass value="${mass_base}" />
+      <inertia ixx="0.001" ixy="0" ixz="0" iyy="0.001" iyz="0" izz="0.001" />
     </inertial>
   </link>
@@ -43,6 +49,10 @@
       </material>
     </visual>
+    <inertial>
+      <mass value="${mass_head}" />
+      <inertia ixx="0.00001" ixy="0" ixz="0" iyy="0.00001" iyz="0" izz="0.00001" />
+    </inertial>
   </link>
-  <!-- Back wheels (cylinders) -->
+  <!-- Back wheels -->
   <link name="left_wheel">
     <visual>
@@ -52,4 +62,8 @@
       <material name="wheel_black" />
     </visual>
+    <inertial>
+      <mass value="${mass_back_wheel}" />
+      <inertia ixx="0.00001" ixy="0" ixz="0" iyy="0.00001" iyz="0" izz="0.00001" />
+    </inertial>
   </link>
   <link name="right_wheel">
@@ -60,21 +74,24 @@
       <material name="wheel_black" />
     </visual>
+    <inertial>
+      <mass value="${mass_back_wheel}" />
+      <inertia ixx="0.00001" ixy="0" ixz="0" iyy="0.00001" iyz="0" izz="0.00001" />
+    </inertial>
   </link>
   <!-- Rotation markers -->
-<link name="left_wheel_marker">
-  <visual>
-    <geometry>
-      <!-- Thin rectangle along the wheel axis -->
-      <box size="${wheel_r*0.2} ${wheel_w * 0.1} ${wheel_r*1.2}" />
-    </geometry>
-    <material name="marker_white">
-      <color rgba="1 1 1 1"/>
-    </material>
-  </visual>
-</link>
+  <link name="left_wheel_marker">
+    <visual>
+      <geometry>
+        <box size="${wheel_r*0.2} ${wheel_w * 0.1} ${wheel_r*1.2}" />
+      </geometry>
+      <material name="marker_white">
+        <color rgba="1 1 1 1" />
+      </material>
+    </visual>
+  </link>
   <link name="right_wheel_marker">
     <visual>
       <geometry>
-        <box size="${wheel_r*1.2} ${wheel_w*0.1} ${wheel_r*0.08}" />
+        <box size="${wheel_r*0.2} ${wheel_w*0.1} ${wheel_r*1.2}" />
       </geometry>
       <material name="marker_white">
@@ -92,6 +109,9 @@
       </material>
     </visual>
+    <inertial>
+      <mass value="${mass_passive_holder}" />
+      <inertia ixx="0.000005" ixy="0" ixz="0" iyy="0.000005" iyz="0" izz="0.000005" />
+    </inertial>
   </link>
-  <!-- Passive wheel as sphere -->
   <link name="passive_wheel">
     <visual>
@@ -101,4 +121,8 @@
       <material name="white" />
     </visual>
+    <inertial>
+      <mass value="${mass_passive_wheel}" />
+      <inertia ixx="0.000002" ixy="0" ixz="0" iyy="0.000002" iyz="0" izz="0.000002" />
+    </inertial>
   </link>
   <!-- ========================== Joints ========================== -->
@@ -120,8 +144,8 @@
   </joint>
   <joint name="left_wheel_marker_fixed" type="fixed">
-  <parent link="left_wheel"/>
-  <child link="left_wheel_marker"/>
-  <origin xyz="0 0 ${-wheel_w / 2}" rpy="${pi/2} 0 ${pi/2}"/>
-</joint>
+    <parent link="left_wheel" />
+    <child link="left_wheel_marker" />
+    <origin xyz="0 0 ${-wheel_w / 2}" rpy="${pi/2} 0 ${pi/2}" />
+  </joint>
   <joint name="base_to_right_wheel" type="continuous">
     <parent link="base_link" />
@@ -133,5 +157,5 @@
     <parent link="right_wheel" />
     <child link="right_wheel_marker" />
-    <origin xyz="0 0 0" rpy="0 0 0" />
+    <origin xyz="0 0 ${wheel_w / 2}" rpy="${pi/2} 0 ${pi/2}" />
   </joint>
   <joint name="base_to_passive_holder" type="fixed">

Commit message: add collisioin

File: urdf/differential_robot.xacro (robot description, xacro)
@@ -11,6 +11,5 @@
   <xacro:property name="head_y" value="0.02" />
   <xacro:property name="head_z" value="0.02" />
-  <xacro:property name="front_wheel_r" value="${(wheel_r - base_thickness/2) / 2}" />
-  <xacro:property name="passive_holder_len" value="0.0006" />
+  <xacro:property name="passive_holder_len" value="0.06" />
   <xacro:property name="passive_wheel_r" value="0.02" />
   <xacro:property name="passive_wheel_w" value="0.01" />
@@ -35,7 +34,12 @@
       </material>
     </visual>
+    <collision>
+      <geometry>
+        <cylinder radius="${base_radius}" length="${base_thickness}" />
+      </geometry>
+    </collision>
     <inertial>
       <mass value="${mass_base}" />
-      <inertia ixx="0.001" ixy="0" ixz="0" iyy="0.001" iyz="0" izz="0.001" />
+      <inertia ixx="0.001" iyy="0.001" izz="0.001" ixy="0" ixz="0" iyz="0"/>
     </inertial>
   </link>
@@ -49,7 +53,12 @@
       </material>
     </visual>
+    <collision>
+      <geometry>
+        <box size="${head_x} ${head_y} ${head_z}" />
+      </geometry>
+    </collision>
     <inertial>
       <mass value="${mass_head}" />
-      <inertia ixx="0.00001" ixy="0" ixz="0" iyy="0.00001" iyz="0" izz="0.00001" />
+      <inertia ixx="0.00001" iyy="0.00001" izz="0.00001" ixy="0" ixz="0" iyz="0"/>
     </inertial>
   </link>
@@ -62,7 +71,12 @@
       <material name="wheel_black" />
     </visual>
+    <collision>
+      <geometry>
+        <cylinder radius="${wheel_r}" length="${wheel_w}" />
+      </geometry>
+    </collision>
     <inertial>
       <mass value="${mass_back_wheel}" />
-      <inertia ixx="0.00001" ixy="0" ixz="0" iyy="0.00001" iyz="0" izz="0.00001" />
+      <inertia ixx="0.00001" iyy="0.00001" izz="0.00001" ixy="0" ixz="0" iyz="0"/>
     </inertial>
   </link>
@@ -74,7 +88,12 @@
       <material name="wheel_black" />
     </visual>
+    <collision>
+      <geometry>
+        <cylinder radius="${wheel_r}" length="${wheel_w}" />
+      </geometry>
+    </collision>
     <inertial>
       <mass value="${mass_back_wheel}" />
-      <inertia ixx="0.00001" ixy="0" ixz="0" iyy="0.00001" iyz="0" izz="0.00001" />
+      <inertia ixx="0.00001" iyy="0.00001" izz="0.00001" ixy="0" ixz="0" iyz="0"/>
     </inertial>
   </link>
@@ -83,5 +102,5 @@
     <visual>
       <geometry>
-        <box size="${wheel_r*0.2} ${wheel_w * 0.1} ${wheel_r*1.2}" />
+        <box size="${wheel_r*0.2} ${wheel_w*0.1} ${wheel_r*1.2}" />
       </geometry>
       <material name="marker_white">
@@ -89,4 +108,9 @@
       </material>
     </visual>
+    <collision>
+      <geometry>
+        <box size="${wheel_r*0.2} ${wheel_w*0.1} ${wheel_r*1.2}" />
+      </geometry>
+    </collision>
   </link>
   <link name="right_wheel_marker">
@@ -99,9 +123,14 @@
       </material>
     </visual>
+    <collision>
+      <geometry>
+        <box size="${wheel_r*0.2} ${wheel_w*0.1} ${wheel_r*1.2}" />
+      </geometry>
+    </collision>
   </link>
   <link name="passive_wheel_holder">
     <visual>
       <geometry>
-        <cylinder radius="${passive_wheel_r}" length="${passive_holder_len}" />
+        <box size="${passive_holder_len} ${passive_wheel_w} ${passive_wheel_w}" />
       </geometry>
       <material name="white">
@@ -109,7 +138,12 @@
       </material>
     </visual>
+    <collision>
+      <geometry>
+        <box size="${passive_holder_len} ${passive_wheel_w} ${passive_wheel_w}" />
+      </geometry>
+    </collision>
     <inertial>
       <mass value="${mass_passive_holder}" />
-      <inertia ixx="0.000005" ixy="0" ixz="0" iyy="0.000005" iyz="0" izz="0.000005" />
+      <inertia ixx="0.000005" iyy="0.000005" izz="0.000005" ixy="0" ixz="0" iyz="0"/>
     </inertial>
   </link>
@@ -119,9 +153,14 @@
         <sphere radius="${passive_wheel_r}" />
       </geometry>
-      <material name="white" />
-    </visual>
+      <material name="wheel_black"/>
+    </visual>
+    <collision>
+      <geometry>
+        <sphere radius="${passive_wheel_r}" />
+      </geometry>
+    </collision>
     <inertial>
       <mass value="${mass_passive_wheel}" />
-      <inertia ixx="0.000002" ixy="0" ixz="0" iyy="0.000002" iyz="0" izz="0.000002" />
+      <inertia ixx="0.000002" iyy="0.000002" izz="0.000002" ixy="0" ixz="0" iyz="0"/>
     </inertial>
   </link>

Commit message: add y axis for wheels

File: urdf/differential_robot.xacro (robot description, xacro)
@@ -41,5 +41,5 @@
     <inertial>
       <mass value="${mass_base}" />
-      <inertia ixx="0.001" iyy="0.001" izz="0.001" ixy="0" ixz="0" iyz="0"/>
+      <inertia ixx="0.001" iyy="0.001" izz="0.001" ixy="0" ixz="0" iyz="0" />
     </inertial>
   </link>
@@ -60,5 +60,5 @@
     <inertial>
       <mass value="${mass_head}" />
-      <inertia ixx="0.00001" iyy="0.00001" izz="0.00001" ixy="0" ixz="0" iyz="0"/>
+      <inertia ixx="0.00001" iyy="0.00001" izz="0.00001" ixy="0" ixz="0" iyz="0" />
     </inertial>
   </link>
@@ -78,5 +78,5 @@
     <inertial>
       <mass value="${mass_back_wheel}" />
-      <inertia ixx="0.00001" iyy="0.00001" izz="0.00001" ixy="0" ixz="0" iyz="0"/>
+      <inertia ixx="0.00001" iyy="0.00001" izz="0.00001" ixy="0" ixz="0" iyz="0" />
     </inertial>
   </link>
@@ -95,5 +95,5 @@
     <inertial>
       <mass value="${mass_back_wheel}" />
-      <inertia ixx="0.00001" iyy="0.00001" izz="0.00001" ixy="0" ixz="0" iyz="0"/>
+      <inertia ixx="0.00001" iyy="0.00001" izz="0.00001" ixy="0" ixz="0" iyz="0" />
     </inertial>
   </link>
@@ -145,5 +145,5 @@
     <inertial>
       <mass value="${mass_passive_holder}" />
-      <inertia ixx="0.000005" iyy="0.000005" izz="0.000005" ixy="0" ixz="0" iyz="0"/>
+      <inertia ixx="0.000005" iyy="0.000005" izz="0.000005" ixy="0" ixz="0" iyz="0" />
     </inertial>
   </link>
@@ -153,5 +153,5 @@
         <sphere radius="${passive_wheel_r}" />
       </geometry>
-      <material name="wheel_black"/>
+      <material name="wheel_black" />
     </visual>
     <collision>
@@ -162,5 +162,5 @@
     <inertial>
       <mass value="${mass_passive_wheel}" />
-      <inertia ixx="0.000002" iyy="0.000002" izz="0.000002" ixy="0" ixz="0" iyz="0"/>
+      <inertia ixx="0.000002" iyy="0.000002" izz="0.000002" ixy="0" ixz="0" iyz="0" />
     </inertial>
   </link>
@@ -176,10 +176,4 @@
     <origin xyz="${base_radius - 0.02} 0 ${base_thickness/2.0 + head_z/2.0}" rpy="0 0 0" />
   </joint>
-  <joint name="base_to_left_wheel" type="continuous">
-    <parent link="base_link" />
-    <child link="left_wheel" />
-    <origin xyz="${-wheel_w/2} ${base_radius + 0.001} 0" rpy="${pi/2} ${pi/2} 0" />
-    <axis xyz="1 0 0" />
-  </joint>
   <joint name="left_wheel_marker_fixed" type="fixed">
     <parent link="left_wheel" />
@@ -187,9 +181,15 @@
     <origin xyz="0 0 ${-wheel_w / 2}" rpy="${pi/2} 0 ${pi/2}" />
   </joint>
+  <joint name="base_to_left_wheel" type="continuous">
+    <parent link="base_link" />
+    <child link="left_wheel" />
+    <origin xyz="${-wheel_w/2} ${base_radius + 0.001} 0" rpy="${pi/2} ${pi/2} 0" />
+    <axis xyz="0 0 1" />
+  </joint>
   <joint name="base_to_right_wheel" type="continuous">
     <parent link="base_link" />
     <child link="right_wheel" />
     <origin xyz="${-wheel_w/2} ${-base_radius} 0" rpy="${pi/2} ${pi/2} 0" />
-    <axis xyz="1 0 0" />
+    <axis xyz="0 0 1" />
   </joint>
   <joint name="right_wheel_marker_fixed" type="fixed">
