Commit message: task 4.2

File: urdf/differential_robot_simu_task4_part2.xacro (robot description, xacro)
@@ -200,5 +200,5 @@
     <parent link="base_link" />
     <child link="left_wheel" />
-    <origin xyz="${-wheel_w/2} ${base_radius + 0.001} 0" rpy="${pi/2} ${pi/2} 0" />
+    <origin xyz="${-wheel_w/2} ${base_radius + 0.001} 0" rpy="${-pi/2} ${pi/2} 0" />
     <axis xyz="0 0 1" />
   </joint>
@@ -206,5 +206,5 @@
     <parent link="base_link" />
     <child link="right_wheel" />
-    <origin xyz="${-wheel_w/2} ${-base_radius} 0" rpy="${pi/2} ${pi/2} 0" />
+    <origin xyz="${-wheel_w/2} ${-base_radius} 0" rpy="${-pi/2} ${pi/2} 0" />
     <axis xyz="0 0 1" />
   </joint>

Commit message: fix robot wheel not appearing

File: urdf/differential_robot_simu_task4_part2.xacro (robot description, xacro)
@@ -224,5 +224,5 @@
     <origin xyz="${base_radius - 0.02} 0 ${-base_thickness/2.0}" rpy="0 0 0" />
   </joint>
-  <joint name="holder_to_passive_wheel" type="continuous">
+  <joint name="holder_to_passive_wheel" type="fixed">
     <parent link="passive_wheel_holder" />
     <child link="passive_wheel" />
