Commit message: add camera working

File: urdf/differential_robot_simu_task6_part2.xacro (robot description, xacro)
@@ -20,4 +20,5 @@
   <xacro:property name="mass_passive_holder" value="0.015" /> <!-- 15g -->
   <xacro:property name="mass_passive_wheel" value="0.01" /> <!-- 10g -->
+  <xacro:property name="camera_size" value="0.05" />
   <material name="wheel_black">
     <color rgba="0.05 0.05 0.05 1.0" />
@@ -186,5 +187,29 @@
     </gazebo>
   </link>
+  <link name="camera_link">
+    <visual>
+      <origin xyz="0 0 0" rpy="0 0 0" />
+      <geometry>
+        <box size="${camera_size} ${camera_size} ${camera_size}" />
+      </geometry>
+      <material name="red" />
+    </visual>
+    <collision>
+      <origin xyz="0 0 0" rpy="0 0 0" />
+      <geometry>
+        <box size="${camera_size} ${camera_size} ${camera_size}" />
+      </geometry>
+    </collision>
+    <inertial>
+      <mass value="0.001" />
+      <inertia ixx="1e-6" iyy="1e-6" izz="1e-6" ixy="0" ixz="0" iyz="0" />
+    </inertial>
+  </link>
   <!-- ========================== Joints ========================== -->
+  <joint name="head_to_camera" type="fixed">
+    <parent link="head_link" />
+    <child link="camera_link" />
+    <origin xyz="0.0 0.0 0.02" rpy="0 0 0" />
+  </joint>
   <joint name="footprint_to_base" type="fixed">
     <parent link="base_footprint" />
@@ -264,3 +289,37 @@
     </plugin>
   </gazebo>
+  <gazebo reference="camera_link">
+    <sensor type="camera" name="camera1">
+      <update_rate>30.0</update_rate>
+      <camera name="head_camera">
+        <horizontal_fov>1.3962634</horizontal_fov>
+        <image>
+          <width>800</width>
+          <height>800</height>
+          <format>R8G8B8</format>
+        </image>
+        <clip>
+          <near>0.02</near>
+          <far>50</far>
+        </clip>
+        <noise>
+          <type>gaussian</type>
+          <mean>0.0</mean>
+          <stddev>0.007</stddev>
+        </noise>
+      </camera>
+      <plugin name="camera_controller" filename="libgazebo_ros_camera.so">
+        <ros>
+          <namespace>/my_robot</namespace>
+        </ros>
+        <alwaysOn>true</alwaysOn>
+        <updateRate>0.0</updateRate>
+        <cameraName>camera1</cameraName>
+        <imageTopicName>/camera1/image_raw</imageTopicName>
+        <cameraInfoTopicName>/camera1/camera_info</cameraInfoTopicName>
+        <frameName>camera_link</frameName>
+        <hackBaseline>0.07</hackBaseline>
+      </plugin>
+    </sensor>
+  </gazebo>
 </robot>
